Commit message: V5 Blocks 2-3: platform random walk; pitched camera, ArUco pad, ground, EGL fixes; CPU-EGL bench

File: v5_shin/assets/lmf2.urdf (robot description, URDF)
Before this commit: robot lmf2, 5 links, 4 joints
Links:
- removed link prop_bl
- removed link prop_br
- removed link prop_fl
- removed link prop_fr
- link base_link: mass 1.2 -> 1.24
Joints:
- removed joint j_bl
- removed joint j_br
- removed joint j_fl
- removed joint j_fr
